File: Schematic/CRW_PCB_v1/CRW_PCB_v1.sch (KiCad schematic (older format))
At the start: 4 parts

Commit message: KiCAD work
Parts:
- removed U?: Teensy4.1, symbol teensy:Teensy4.1
- removed U?: BNO055, Package_LGA:LGA-28_5.2x3.8mm_P0.5mm, symbol Sensor_Motion:BNO055
- removed U?: BMP388, symbol Sensor_Pressure:BMP388
- removed U?: VL53L1CXV0FY1, Sensor_Distance:ST_VL53L1x, symbol Sensor_Distance:VL53L1CXV0FY1
- added U?: BMP388, PQFN50P200X200X80-10N, symbol BMP388:BMP388
- added U?: BNO055, LGA28R50P4X10_380X520X100, symbol BNO055:BNO055
- added U?: DEV-16771, DEV-16771, symbol DEV-16771:DEV-16771
Changed lines of the file:
@@
 $EndDescr
 $Comp
-L teensy:Teensy4.1 U?
-U 1 1 5FD1783C
-P 900 -2600
-F 0 "U?" H 900 -35 50  0000 C CNN
-F 1 "Teensy4.1" H 900 -126 50  0000 C CNN
-F 2 "" H 500 -2200 50  0001 C CNN
-F 3 "" H 500 -2200 50  0001 C CNN
-	1    900  -2600
+L BMP388:BMP388 U?
+U 1 1 5FDD1DDB
+P 5100 1850
+F 0 "U?" H 5100 2617 50  0000 C CNN
+F 1 "BMP388" H 5100 2526 50  0000 C CNN
+F 2 "PQFN50P200X200X80-10N" H 5100 1850 50  0001 L BNN
+F 3 "" H 5100 1850 50  0001 L BNN
+F 4 "1.1" H 5100 1850 50  0001 L BNN "PARTREV"
+F 5 "BOSCH" H 5100 1850 50  0001 L BNN "MANUFACTURER"
+F 6 "IPC 7351B" H 5100 1850 50  0001 L BNN "STANDARD"
+	1    5100 1850
 	1    0    0    -1
 $EndComp
 $Comp
-L Sensor_Motion:BNO055 U?
-U 1 1 5FD29B92
-P 6500 -4400
-F 0 "U?" H 6500 -3519 50  0000 C CNN
-F 1 "BNO055" H 6500 -3610 50  0000 C CNN
-F 2 "Package_LGA:LGA-28_5.2x3.8mm_P0.5mm" H 6750 -5050 50  0001 L CNN
-F 3 "https://ae-bst.resource.bosch.com/media/_tech/media/datasheets/BST_BNO055_DS000_14.pdf" H 6500 -4200 50  0001 C CNN
-	1    6500 -4400
+L BNO055:BNO055 U?
+U 1 1 5FDD292B
+P 8950 2200
+F 0 "U?" H 8950 2967 50  0000 C CNN
+F 1 "BNO055" H 8950 2876 50  0000 C CNN
+F 2 "LGA28R50P4X10_380X520X100" H 8950 2200 50  0001 L BNN
+F 3 "" H 8950 2200 50  0001 L BNN
+F 4 "BOSCH" H 8950 2200 50  0001 L BNN "MANUFACTURER"
+	1    8950 2200
 	1    0    0    -1
 $EndComp
 $Comp
-L Sensor_Pressure:BMP388 U?
-U 1 1 5FD30692
-P 6000 -2150
-F 0 "U?" H 6500 -869 50  0000 C CNN
-F 1 "BMP388" H 6500 -960 50  0000 C CNN
-F 2 "" H 6500 -1650 50  0001 C CNN
-F 3 "" H 6500 -1650 50  0001 C CNN
-	1    6000 -2150
+L DEV-16771:DEV-16771 U?
+U 1 1 5FDD3AD4
+P 2000 4300
+F 0 "U?" H 2000 6267 50  0000 C CNN
+F 1 "DEV-16771" H 2000 6176 50  0000 C CNN
+F 2 "DEV-16771" H 2000 4300 50  0001 L BNN
+F 3 "" H 2000 4300 50  0001 L BNN
+F 4 "Evaluation Boards - Embedded - MCU, DSP" H 2000 4300 50  0001 L BNN "CATEGORIES"
+F 5 "SparksFun" H 2000 4300 50  0001 L BNN "MANUFACTURER"
+	1    2000 4300
 	1    0    0    -1
 $EndComp
-$Comp
-L Sensor_Distance:VL53L1CXV0FY1 U?
-U 1 1 5FD335B3
-P -950 -5450
-F 0 "U?" H -620 -5404 50  0000 L CNN
-F 1 "VL53L1CXV0FY1" H -620 -5495 50  0000 L CNN
-F 2 "Sensor_Distance:ST_VL53L1x" H -275 -6000 50  0001 C CNN
-F 3 "https://www.st.com/resource/en/datasheet/vl53l1x.pdf" H -850 -5450 50  0001 C CNN
-	1    -950 -5450
-	1    0    0    -1
-$EndComp

Commit message: Schematic work
Parts:
- added BT1: 1048P, BAT_1048P, symbol 1048P:1048P
- added Cff1, Cff2: 6.8pF, symbol Device:C
- added Ci1, Ci2: 10uF, symbol Device:C
- added Co1, Co2: 22uF, symbol Device:C
- added L1, L2: 10uH, symbol Device:L
- added R1: 560k, symbol Device:R
- added R10, R3, R4, R9: 1M, symbol Device:R
- added R11: 820k, symbol Device:R
- added R12: 91k, symbol Device:R
- added R2, R6, R8: 100k, symbol Device:R
- added R5, R7: 130k, symbol Device:R
- added U2, U6: TPS62051DGS, CRW_PCB_v1:TPS62051DGS_VSSOP, symbol CRW_PCB_v1:TPS62051DGS
- added XBEE1: XBEE Wire, DIP2200W51P200L3294H279Q20P, symbol XBP9B-DMWT-002:XBP9B-DMWT-002
- MCU1: renamed from U?; value DEV-16771 -> TEENSY 4.1
- gave numbers to parts that had none: 2
Connections:
- net labels added: +3V3, +5V, +BATT, -BATT
- wire segments 0 -> 115
Other:
- note added: "3.3V Regulator"
- note added: "5V Regulator"

Commit message: More Schematic Work
Parts:
- added C1, C2, C5: 100nF, symbol Device:C
- added C3: 1uF, symbol Device:C
- added C4: 120nF, symbol Device:C
- added CAM1, CAM2, CAM3: CAMERA, symbol Connector:Conn_01x06_Female
- added D1: D_Zener, symbol Device:D_Zener
- added J1: SWITCH, symbol Connector:Conn_01x02_Female
- added Q1: Q_PMOS_GSD, symbol Device:Q_PMOS_GSD
- added R14, R15, R16, R17, R18, R5: 10k, symbol Device:R
- added R19, R20, R21: R, symbol Device:R
- added TH1: Thermistor, symbol Device:Thermistor
- renumbered BT1 to BAT1, R5 to R1, R1 to R10, R2 to R11, R11 to R12, R12 to R13, R6 to R2, R7 to R3, R8 to R4, R3 to R6, R9 to R7, R4 to R8, R10 to R9, U2 to U1, U6 to U2
Connections:
- net labels added: +3.3V, BATT_ADC, BMP_INT, BMP_SS, CAM1_SS, CAM2_SS, CAM3_SS, FROM_SW, I2C_SCL, I2C_SDA, IMU_ADDR_SEL, IMU_INT, IMU_~RESET, SPI_MISO, SPI_MOSI, SPI_SCLK, THERM_ADC, TO_SW, XBEE_UART_MISO, XBEE_UART_MOSI, XBEE_~RESET
- wire segments 115 -> 227
- no-connect marks 0 -> 36
Other:
- note added: "BMP"
- note added: "Batteries"
- note added: "IMU"
- note added: "Power Systems"
- note added: "Reverse Polarity Protection"
- note added: "XBEE"
- moved on the sheet: Cff1, Cff2, Ci1, Ci2, Co1, Co2, L1, L2, R1, R10, R11, R12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

Commit message: Finished Schematic
Parts:
- removed BAT1: 1048P, BAT_1048P, symbol 1048P:1048P
- added C1, C2, C3, C4, C5, C6: 0.1uF, symbol Device:C
- added D2, D3: D_Schottky, symbol Device:D_Schottky
- added D4: FLYBACK, symbol Device:D
- added J2: LEVEL1, symbol Connector:Conn_01x02_Female
- added J3: AUTOGYRO_RELEASE, symbol Connector:Conn_01x02_Female
- added J4: GPS_Connector, symbol Connector:Conn_01x03_Female
- added J5: LEVEL2, symbol Connector:Conn_01x02_Female
- added J6: QWIIC_Connector, symbol Connector:Conn_01x04_Female
- added J7: LEVEL3, symbol Connector:Conn_01x02_Female
- added Q2: Q_PMOS_GSD, symbol Device:Q_PMOS_GSD
- added Q3, Q4: Q_NMOS_GSD, symbol Device:Q_NMOS_GSD
- added R10, R16, R17, R18, R22, R26: 10k, symbol Device:R
- added R15, R23: 220, symbol Device:R
- added R19, R20, R21: 4.7k, symbol Device:R
- added U3, U4, U5: DRV8838DSGR, CRW_PCB_v1:DRV8838DSGR, symbol CRW_PCB_v1:DRV8838DSGR
- J1: value SWITCH -> BATTERIES
- MCU1: footprint DEV-16771 -> Teensy4_1:DEV-16771
- R24: renamed from R14; value 10k -> 4.7k
- R25: renamed from R19; value R -> 50k
- R28: renamed from R16; value 10k -> 4.7k
- R30: renamed from R20; value R -> 100k
- R31: renamed from R21; value R -> 50k
- U6: renamed from U3; footprint PQFN50P200X200X80-10N -> BMP388:PQFN50P200X200X80-10N
- U7: renamed from U4; footprint LGA28R50P4X10_380X520X100 -> BNO055:LGA28R50P4X10_380X520X100
- XBEE1: footprint DIP2200W51P200L3294H279Q20P -> XBEE:DIP2200W51P200L3294H279Q20P
- renumbered C4 to C10, C5 to C11, C1 to C7, C3 to C8, C2 to C9, R5 to R1, R10 to R11, R11 to R12, R12 to R13, R13 to R14, R1 to R2, R15 to R27, R17 to R29, R2 to R3, R18 to R32, R3 to R4, R4 to R5
Connections:
- net labels added: BMP_ADDR_SEL, CAM_PWR, GPS_UART_MISO, GYRO_RELEASE, LEVEL1_DIR, LEVEL1_PWM, LEVEL1_~SLEEP, LEVEL2_DIR, LEVEL2_PWM, LEVEL2_~SLEEP, LEVEL3_DIR, LEVEL3_PWM, LEVEL3_~SLEEP, USB_PWR
- net labels removed: BMP_SS, FROM_SW, TO_SW
- wire segments 227 -> 346
- no-connect marks 36 -> 49
Other:
- note added: "Battery Voltage"
- note added: "Cameras"
- note added: "GPS"
- note added: "Motor Drivers"
- note added: "Notation Clarification (so I don't have to change everything)\n+BATT is the driving voltage of the load\n-BATT is GND\nUSB_PWR is the connected USB's voltage input (GND when not connected)"
- note added: "Pressure"
- note added: "Rangefinder"
- note added: "Release"
- note added: "SPI Chip Select Pull-Ups"
- note added: "Source Switching"
- note added: "Thermistor"
- note removed: "BMP"
- note removed: "Batteries"
- moved on the sheet: C7, C9, D1, J1, MCU1, Q1, R1, R25, R30, R31, TH1, U6

Commit message: Removed .lib from .gitignore
Parts:
- removed J1: BATTERIES, symbol Connector:Conn_01x02_Female
- added J1: BATTERIES, Connector_JST:JST_SH_BM02B-SRSS-TB_1x02-1MP_P1.00mm_Vertical, symbol Connector:Conn_01x02_Male
- C1, C10, C2, C3, C4, C5, C6, C8: footprint (none) -> Capacitor_SMD:C_0603_1608Metric_Pad1.08x0.95mm_HandSolder
- C11, C7, C9: value 100nF -> 0.1uF; footprint (none) -> Capacitor_SMD:C_0603_1608Metric_Pad1.08x0.95mm_HandSolder
- CAM1, CAM2, CAM3: footprint (none) -> Connector_JST:JST_SH_BM06B-SRSS-TB_1x06-1MP_P1.00mm_Vertical
- Cff1, Cff2: footprint (none) -> Capacitor_SMD:C_0402_1005Metric_Pad0.74x0.62mm_HandSolder
- Ci1, Ci2, Co1, Co2: footprint (none) -> Capacitor_SMD:C_0805_2012Metric_Pad1.18x1.45mm_HandSolder
- D1: footprint (none) -> Diode_SMD:D_SOD-123
- D2, D3: footprint (none) -> Diode_SMD:D_SMB
- D4: footprint (none) -> Diode_SMD:D_SMC
- J2, J3, J5, J7: footprint (none) -> Connector_JST:JST_SH_BM02B-SRSS-TB_1x02-1MP_P1.00mm_Vertical
- J4: footprint (none) -> Connector_JST:JST_SH_BM03B-SRSS-TB_1x03-1MP_P1.00mm_Vertical
- J6: footprint (none) -> Connector_JST:JST_SH_BM04B-SRSS-TB_1x04-1MP_P1.00mm_Vertical
- L1, L2: footprint (none) -> Inductor_SMD:L_Taiyo-Yuden_NR-60xx
- Q1, Q2, Q3, Q4: footprint (none) -> Package_TO_SOT_SMD:SC-59_Handsoldering
- R1, R10, R11, R12, R13, R14, R16, R17, R18, R19, R2, R20, R21, R22, R24, R26, R27, R28, R29, R3, R30, R32, R4, R5, R6, R7, R8, R9: footprint (none) -> Resistor_SMD:R_0402_1005Metric_Pad0.72x0.64mm_HandSolder
- R15, R23: footprint (none) -> Resistor_SMD:R_0603_1608Metric_Pad0.98x0.95mm_HandSolder
- R25, R31: value 50k -> 47k; footprint (none) -> Resistor_SMD:R_0402_1005Metric_Pad0.72x0.64mm_HandSolder
- TH1: footprint (none) -> Resistor_THT:R_Axial_DIN0204_L3.6mm_D1.6mm_P2.54mm_Vertical
Connections:
- net -BATT: now also C3.2, C4.2, C5.2, C6.2, U4.4 (GND), U5.4 (GND), J1.2 (Pin_2)
- net at U3.2 (OUT1): now also J2.2 (Pin_2); no longer J2.1 (Pin_1)
- net at U3.3 (OUT2): now also J2.1 (Pin_1); no longer J2.2 (Pin_2)
- net at U4.2 (OUT1): now also J5.2 (Pin_2); no longer J5.1 (Pin_1)
- net at U4.3 (OUT2): now also J5.1 (Pin_1); no longer J5.2 (Pin_2)
- net at U5.2 (OUT1): now also J7.2 (Pin_2); no longer J7.1 (Pin_1)
- net at U5.3 (OUT2): now also J7.1 (Pin_1); no longer J7.2 (Pin_2)
- net at Q1.3 (D): now also J1.1 (Pin_1)

Commit message: Maybe Finished PCB
Connections:
- net -BATT: now also U3.9 (TP), U4.9 (TP), U5.9 (TP)
Changed lines of the file:
@@
 Wire Wire Line
 	7200 11450 7250 11450
+Wire Wire Line
+	7250 11350 7200 11350
+Wire Wire Line
+	7200 11350 7200 11450
+Wire Wire Line
+	4050 11350 4000 11350
+Wire Wire Line
+	4000 11350 4000 11450
+Wire Wire Line
+	600  11350 550  11350
+Wire Wire Line
+	550  11350 550  11450
 $EndSCHEMATC

Commit message: Change Power connectors
Parts:
- BATT1: renamed from J1; footprint Connector_JST:JST_SH_BM02B-SRSS-TB_1x02-1MP_P1.00mm_Vertical -> Connector_JST:JST_PH_B2B-PH-K_1x02_P2.00mm_Vertical
- RELEASE1: renamed from J3; footprint Connector_JST:JST_SH_BM02B-SRSS-TB_1x02-1MP_P1.00mm_Vertical -> Connector_JST:JST_PH_B2B-PH-K_1x02_P2.00mm_Vertical
- renumbered U7 to BMP1, U6 to BNO1, J4 to GPS1, J2 to MOTOR1, J5 to MOTOR2, J7 to MOTOR3, J6 to RANGE1
Connections:
- no-connect marks 49 -> 33
Other:
- note added: "Notation Clarification\n+BATT is the driving voltage of the load\n-BATT is GND\nUSB_PWR is the connected USB's voltage input (GND when not connected)"
- note removed: "Notation Clarification (so I don't have to change everything)\n+BATT is the driving voltage of the load\n-BATT is GND\nUSB_PWR is the connected USB's voltage input (GND when not connected)"
Changed lines of the file:
@@
 	14000 2325 14000 2375
 $Comp
-L BNO055:BNO055 U7
+L BNO055:BNO055 BMP1
 U 1 1 5FDD292B
 P 14850 1375
-F 0 "U7" H 14850 2142 50  0000 C CNN
+F 0 "BMP1" H 14850 2142 50  0000 C CNN
 F 1 "BNO055" H 14850 2051 50  0000 C CNN
 F 2 "BNO055:LGA28R50P4X10_380X520X100" H 14850 1375 50  0001 L BNN
@@
 NoConn ~ 3500 2100
 NoConn ~ 1700 3300
-NoConn ~ 2800 4700
-NoConn ~ 2700 4700
-NoConn ~ 2600 4700
-NoConn ~ 2500 4700
-NoConn ~ 2400 4700
-NoConn ~ 1700 1150
-NoConn ~ 1700 1250
-NoConn ~ 1700 1350
-NoConn ~ 1700 1450
-NoConn ~ 1700 1550
-NoConn ~ 1700 1650
-NoConn ~ 3500 1550
-NoConn ~ 3500 1450
-NoConn ~ 3500 1350
-NoConn ~ 3500 1250
-NoConn ~ 3500 1150
-$Comp
-L BMP388:BMP388 U6
+$Comp
+L BMP388:BMP388 BNO1
 U 1 1 5FDD1DDB
 P 13150 6650
-F 0 "U6" H 13150 7417 50  0000 C CNN
+F 0 "BNO1" H 13150 7417 50  0000 C CNN
 F 1 "BMP388" H 13150 7326 50  0000 C CNN
 F 2 "BMP388:PQFN50P200X200X80-10N" H 13150 6650 50  0001 L BNN
@@
 Cameras
 $Comp
-L Connector:Conn_01x04_Female J6
+L Connector:Conn_01x04_Female RANGE1
 U 1 1 606C4571
 P 7350 9500
-F 0 "J6" V 7500 9550 50  0000 R CNN
+F 0 "RANGE1" V 7500 9550 50  0000 R CNN
 F 1 "QWIIC_Connector" V 7400 9800 50  0000 R CNN
 F 2 "Connector_JST:JST_SH_BM04B-SRSS-TB_1x04-1MP_P1.00mm_Vertical" H 7350 9500 50  0001 C CNN
@@
 GPS_UART_MISO
 $Comp
-L Connector:Conn_01x03_Female J4
+L Connector:Conn_01x03_Female GPS1
 U 1 1 6072A007
 P 4050 9300
-F 0 "J4" V 4200 9350 50  0000 R CNN
+F 0 "GPS1" V 4200 9350 50  0000 R CNN
 F 1 "GPS_Connector" V 4100 9550 50  0000 R CNN
 F 2 "Connector_JST:JST_SH_BM03B-SRSS-TB_1x03-1MP_P1.00mm_Vertical" H 4050 9300 50  0001 C CNN
@@
 Connection ~ 200  11450
 $Comp
-L Connector:Conn_01x02_Female J2
+L Connector:Conn_01x02_Female MOTOR1
 U 1 1 600AC24E
 P 1500 11750
-F 0 "J2" V 1438 11562 50  0000 R CNN
+F 0 "MOTOR1" V 1438 11562 50  0000 R CNN
 F 1 "LEVEL1" V 1347 11562 50  0000 R CNN
 F 2 "Connector_JST:JST_SH_BM02B-SRSS-TB_1x02-1MP_P1.00mm_Vertical" H 1500 11750 50  0001 C CNN
@@
 Connection ~ 3650 11450
 $Comp
-L Connector:Conn_01x02_Female J5
+L Connector:Conn_01x02_Female MOTOR2
 U 1 1 6012744B
 P 4950 11750
-F 0 "J5" V 4888 11562 50  0000 R CNN
+F 0 "MOTOR2" V 4888 11562 50  0000 R CNN
 F 1 "LEVEL2" V 4797 11562 50  0000 R CNN
 F 2 "Connector_JST:JST_SH_BM02B-SRSS-TB_1x02-1MP_P1.00mm_Vertical" H 4950 11750 50  0001 C CNN
@@
 Connection ~ 6850 11450
 $Comp
-L Connector:Conn_01x02_Female J7
+L Connector:Conn_01x02_Female MOTOR3
 U 1 1 6013C77C
 P 8150 11750
-F 0 "J7" V 8088 11562 50  0000 R CNN
+F 0 "MOTOR3" V 8088 11562 50  0000 R CNN
 F 1 "LEVEL3" V 7997 11562 50  0000 R CNN
 F 2 "Connector_JST:JST_SH_BM02B-SRSS-TB_1x02-1MP_P1.00mm_Vertical" H 8150 11750 50  0001 C CNN
@@
 CAM_PWR
 $Comp
-L Connector:Conn_01x02_Female J3
+L Connector:Conn_01x02_Female RELEASE1
 U 1 1 5FE6CB20
 P 1750 9100
-F 0 "J3" V 1900 9150 50  0000 R CNN
+F 0 "RELEASE1" V 1900 9150 50  0000 R CNN
 F 1 "AUTOGYRO_RELEASE" V 1800 9450 50  0000 R CNN
-F 2 "Connector_JST:JST_SH_BM02B-SRSS-TB_1x02-1MP_P1.00mm_Vertical" H 1750 9100 50  0001 C CNN
+F 2 "Connector_JST:JST_PH_B2B-PH-K_1x02_P2.00mm_Vertical" H 1750 9100 50  0001 C CNN
 F 3 "~" H 1750 9100 50  0001 C CNN
 	1    1750 9100
@@
 	-1   0    0    1
 $EndComp
-Text Notes -5000 -700 0    50   ~ 0
-Notation Clarification (so I don't have to change everything)\n+BATT is the driving voltage of the load\n-BATT is GND\nUSB_PWR is the connected USB's voltage input (GND when not connected)
+Text Notes -4600 2050 0    50   ~ 0
+Notation Clarification\n+BATT is the driving voltage of the load\n-BATT is GND\nUSB_PWR is the connected USB's voltage input (GND when not connected)
 Wire Wire Line
 	3700 1900 3500 1900
@@
 $EndComp
 $Comp
-L Connector:Conn_01x02_Male J1
+L Connector:Conn_01x02_Male BATT1
 U 1 1 5FF7185A
 P -4300 100
-F 0 "J1" V -4238 144 50  0000 L CNN
+F 0 "BATT1" V -4238 144 50  0000 L CNN
 F 1 "BATTERIES" V -4147 144 50  0000 L CNN
-F 2 "Connector_JST:JST_SH_BM02B-SRSS-TB_1x02-1MP_P1.00mm_Vertical" H -4300 100 50  0001 C CNN
+F 2 "Connector_JST:JST_PH_B2B-PH-K_1x02_P2.00mm_Vertical" H -4300 100 50  0001 C CNN
 F 3 "~" H -4300 100 50  0001 C CNN
 	1    -4300 100

Commit message: Used Hierarchical Sheets
Parts:
- removed BATT1: BATTERIES, Connector_JST:JST_PH_B2B-PH-K_1x02_P2.00mm_Vertical, symbol Connector:Conn_01x02_Male
- removed BMP1: BNO055, BNO055:LGA28R50P4X10_380X520X100, symbol BNO055:BNO055
- removed BNO1: BMP388, BMP388:PQFN50P200X200X80-10N, symbol BMP388:BMP388
- removed C1, C11, C2, C3, C4, C5, C6, C7, C9: 0.1uF, Capacitor_SMD:C_0603_1608Metric_Pad1.08x0.95mm_HandSolder, symbol Device:C
- removed C10: 120nF, Capacitor_SMD:C_0603_1608Metric_Pad1.08x0.95mm_HandSolder, symbol Device:C
- removed C8: 1uF, Capacitor_SMD:C_0603_1608Metric_Pad1.08x0.95mm_HandSolder, symbol Device:C
- removed CAM1, CAM2, CAM3: CAMERA, Connector_JST:JST_SH_BM06B-SRSS-TB_1x06-1MP_P1.00mm_Vertical, symbol Connector:Conn_01x06_Female
- removed Cff1, Cff2: 6.8pF, Capacitor_SMD:C_0402_1005Metric_Pad0.74x0.62mm_HandSolder, symbol Device:C
- removed Ci1, Ci2: 10uF, Capacitor_SMD:C_0805_2012Metric_Pad1.18x1.45mm_HandSolder, symbol Device:C
- removed Co1, Co2: 22uF, Capacitor_SMD:C_0805_2012Metric_Pad1.18x1.45mm_HandSolder, symbol Device:C
- removed D1: D_Zener, Diode_SMD:D_SOD-123, symbol Device:D_Zener
- removed D2, D3: D_Schottky, Diode_SMD:D_SMB, symbol Device:D_Schottky
- removed D4: FLYBACK, Diode_SMD:D_SMC, symbol Device:D
- removed GPS1: GPS_Connector, Connector_JST:JST_SH_BM03B-SRSS-TB_1x03-1MP_P1.00mm_Vertical, symbol Connector:Conn_01x03_Female
- removed L1, L2: 10uH, Inductor_SMD:L_Taiyo-Yuden_NR-60xx, symbol Device:L
- removed MOTOR1: LEVEL1, Connector_JST:JST_SH_BM02B-SRSS-TB_1x02-1MP_P1.00mm_Vertical, symbol Connector:Conn_01x02_Female
- removed MOTOR2: LEVEL2, Connector_JST:JST_SH_BM02B-SRSS-TB_1x02-1MP_P1.00mm_Vertical, symbol Connector:Conn_01x02_Female
- removed MOTOR3: LEVEL3, Connector_JST:JST_SH_BM02B-SRSS-TB_1x02-1MP_P1.00mm_Vertical, symbol Connector:Conn_01x02_Female
- removed Q1, Q2: Q_PMOS_GSD, Package_TO_SOT_SMD:SC-59_Handsoldering, symbol Device:Q_PMOS_GSD
- removed Q3, Q4: Q_NMOS_GSD, Package_TO_SOT_SMD:SC-59_Handsoldering, symbol Device:Q_NMOS_GSD
- removed R1, R10, R16, R17, R18, R22, R26, R29, R32: 10k, Resistor_SMD:R_0402_1005Metric_Pad0.72x0.64mm_HandSolder, symbol Device:R
- removed R11: 560k, Resistor_SMD:R_0402_1005Metric_Pad0.72x0.64mm_HandSolder, symbol Device:R
- removed R12, R3, R30, R5: 100k, Resistor_SMD:R_0402_1005Metric_Pad0.72x0.64mm_HandSolder, symbol Device:R
- removed R13: 820k, Resistor_SMD:R_0402_1005Metric_Pad0.72x0.64mm_HandSolder, symbol Device:R
- removed R14: 91k, Resistor_SMD:R_0402_1005Metric_Pad0.72x0.64mm_HandSolder, symbol Device:R
- removed R15, R23: 220, Resistor_SMD:R_0603_1608Metric_Pad0.98x0.95mm_HandSolder, symbol Device:R
- removed R19, R20, R21, R24, R28: 4.7k, Resistor_SMD:R_0402_1005Metric_Pad0.72x0.64mm_HandSolder, symbol Device:R
- removed R2, R4: 130k, Resistor_SMD:R_0402_1005Metric_Pad0.72x0.64mm_HandSolder, symbol Device:R
- removed R25, R31: 47k, Resistor_SMD:R_0402_1005Metric_Pad0.72x0.64mm_HandSolder, symbol Device:R
- removed R6, R7, R8, R9: 1M, Resistor_SMD:R_0402_1005Metric_Pad0.72x0.64mm_HandSolder, symbol Device:R
- removed RANGE1: QWIIC_Connector, Connector_JST:JST_SH_BM04B-SRSS-TB_1x04-1MP_P1.00mm_Vertical, symbol Connector:Conn_01x04_Female
- removed RELEASE1: AUTOGYRO_RELEASE, Connector_JST:JST_PH_B2B-PH-K_1x02_P2.00mm_Vertical, symbol Connector:Conn_01x02_Female
- removed TH1: Thermistor, Resistor_THT:R_Axial_DIN0204_L3.6mm_D1.6mm_P2.54mm_Vertical, symbol Device:Thermistor
- removed U1, U2: TPS62051DGS, CRW_PCB_v1:TPS62051DGS_VSSOP, symbol CRW_PCB_v1:TPS62051DGS
- removed U3, U4, U5: DRV8838DSGR, CRW_PCB_v1:DRV8838DSGR, symbol CRW_PCB_v1:DRV8838DSGR
Connections:
- no-connect marks 33 -> 28
Other:
- note removed: "3.3V Regulator"
- note removed: "5V Regulator"
- note removed: "Battery Voltage"
- note removed: "Cameras"
- note removed: "GPS"
- note removed: "IMU"
- note removed: "Motor Drivers"
- note removed: "Notation Clarification\n+BATT is the driving voltage of the load\n-BATT is GND\nUSB_PWR is the connected USB's voltage input (GND when not connected)"
- note removed: "Power Systems"
- note removed: "Pressure"
- note removed: "Rangefinder"
- note removed: "Release"
- note removed: "Reverse Polarity Protection"
- note removed: "SPI Chip Select Pull-Ups"
- note removed: "Source Switching"
- note removed: "Thermistor"
- moved on the sheet: R27, XBEE1
